Commit message: Fixed Descartes + IKFast for the ABB IRB2600

File: abb_irb2600_trispector_support/urdf/abb_irb2600_trispector_macro.xacro (robot description, xacro)
@@ -1,4 +1,5 @@
 <?xml version="1.0" ?>
-<robot name="abb_irb2600_trispector" xmlns:xacro="http://ros.org/wiki/xacro">
+<robot xmlns:xacro="http://ros.org/wiki/xacro">
+    <xacro:macro name="abb_irb2600_trispector" params="prefix">
     <xacro:include filename="$(find abb_irb2600_support)/urdf/irb2600_12_165_macro.xacro" />
     <xacro:include filename="$(find trispector_1060_support)/urdf/trispector_macro.xacro" />
@@ -14,9 +15,9 @@
         <origin xyz="0.0 0.0 0.0" rpy="-1.5708 -1.5708 0.0" />
     </joint>
-    <joint name="world_to_robot" type="fixed">
+    <!-- <joint name="world_to_robot" type="fixed">
         <parent link="world" />
         <child link="base_link" />
         <origin xyz="0.0 0.0 0.0" rpy="0.0 0.0 0.0" />
-    </joint>
+    </joint> -->
     <joint name="world_to_camera" type="fixed">
         <parent link="world" />
@@ -24,3 +25,4 @@
         <origin xyz="-0.25 -0.5 1.25" rpy="0.0 3.14159 0.0" />
     </joint>
+    </xacro:macro>
 </robot>

File: myworkcell_support/urdf/workcell.urdf (robot description, URDF)
Before this commit: robot myworkcell, 17 links, 16 joints
Links:
- removed link eff_frame
- removed link laser_area
- removed link scan_area
- removed link scan_area_origin
- removed link tcp
- removed link trispector
- added link ee_base; collision mesh filename=package://myworkcell_support/meshes/puzzle_mount.stl; visual mesh filename=package://myworkcell_support/meshes/puzzle_mount.stl
- added link ee_mount
- added link grinder_frame; collision mesh filename=package://myworkcell_support/meshes/grinder_collision.dae; visual mesh filename=package://myworkcell_support/meshes/grinder_visual.dae
- added link part; collision mesh filename=package://myworkcell_support/meshes/puzzle_bent.dae; visual mesh filename=package://myworkcell_support/meshes/puzzle_bent.dae
- added link tool1
Joints:
- removed joint eff_frame_to_trispector
- removed joint joint_scan_area_origin
- removed joint joint_tcp
- removed joint origin_to_laser_area
- removed joint origin_to_scan_area
- removed joint robot_to_eff
- added joint ee_base-tool1: type fixed, parent ee_base, child tool1, origin xyz=-0.0083 0.0541 0.0143 rpy=0.523599 -0.523599 0
- added joint ee_mount-ee_base: type fixed, parent ee_mount, child ee_base, origin xyz=0 0 0 rpy=0 0 0
- added joint tool1-part: type fixed, parent tool1, child part, origin xyz=0.0110 0.0030 -0.0379 rpy=0 -0.2618 0
- added joint tool_to_puzzle: type fixed, parent tool0, child ee_mount, origin xyz=0 0 0 rpy=1.5708 0 0
- added joint world_to_grinder: type fixed, parent world, child grinder_frame, origin xyz=0.0 -0.4 0.1 rpy=0 3.14159 0

File: myworkcell_support/urdf/workcell.xacro (robot description, xacro)
@@ -1,26 +1,38 @@
 <?xml version="1.0" ?>
 <robot name="myworkcell" xmlns:xacro="http://ros.org/wiki/xacro">
-    <xacro:include filename="$(find abb_irb2600_support)/urdf/irb2600_12_165_macro.xacro" />
-    <xacro:include filename="$(find trispector_1060_support)/urdf/trispector_macro.xacro" />
-    <xacro:abb_irb2600_12_165 prefix="" />
-    <xacro:trispector prefix="" />
+  <xacro:include filename="$(find abb_irb2600_support)/urdf/irb2600_12_165_macro.xacro" />
+  <!-- <xacro:include filename="$(find trispector_1060_support)/urdf/trispector_macro.xacro" /> -->
+  <xacro:include filename="$(find myworkcell_support)/urdf/grinder.xacro" />
+  <xacro:include filename="$(find myworkcell_support)/urdf/puzzle_mount.xacro" />
 <!-- Links -->
-    <link name="world" />
-    <link name="camera_frame" />
+  <link name="world" />
+  <link name="camera_frame" />
+  <xacro:abb_irb2600_12_165 prefix="" />
+  <!-- <xacro:trispector prefix="" /> -->
 <!-- Joints -->
-    <joint name="robot_to_eff" type="fixed">
-        <parent link="tool0" />
-        <child link="eff_frame" />
-        <origin xyz="0.0 0.0 0.0" rpy="-1.5708 -1.5708 0.0" />
-    </joint>
-    <joint name="world_to_robot" type="fixed">
-        <parent link="world" />
-        <child link="base_link" />
-        <origin xyz="0.0 0.0 0.0" rpy="0.0 0.0 0.0" />
-    </joint>
-    <joint name="world_to_camera" type="fixed">
-        <parent link="world" />
-        <child link="camera_frame" />
-        <origin xyz="-0.25 -0.5 1.25" rpy="0.0 3.14159 0.0" />
-    </joint>
+  <joint name="world_to_camera" type="fixed">
+    <parent link="world" />
+    <child link="camera_frame" />
+    <origin xyz="-0.25 -0.5 1.25" rpy="0.0 3.14159 0.0" />
+  </joint>
+  <joint name="world_to_robot" type="fixed">
+    <parent link="world" />
+    <child link="base_link" />
+    <origin xyz="0.0 0.0 0.0" rpy="0.0 0.0 0.0" />
+  </joint>
+  <joint name="world_to_grinder" type="fixed">
+    <parent link="world" />
+    <child link="grinder_frame" />
+    <origin xyz="0.0 -0.8 0.1" rpy="0 3.14159 0"/>
+  </joint>
+  <joint name="tool_to_puzzle" type="fixed">
+    <parent link="tool0" />
+    <child link="ee_mount" />
+    <origin xyz="0 0 0" rpy="1.5708 0 0"/>
+  </joint>
+  <!-- <joint name="robot_to_eff" type="fixed">
+    <parent link="tool0" />
+    <child link="eff_frame" />
+    <origin xyz="0.0 0.0 0.0" rpy="-1.5708 -1.5708 0.0" />
+  </joint> -->
 </robot>

Commit message: Added ABB IRBT-2005 track

File: abb_irb2600_trispector_support/urdf/abb_irb2600_trispector_macro.xacro (robot description, xacro)
@@ -7,6 +7,6 @@
     <xacro:trispector prefix="" />
 <!-- Links -->
-    <link name="world" />
-    <link name="camera_frame" />
+    <!-- <link name="world" />
+    <link name="camera_frame" /> -->
 <!-- Joints -->
     <joint name="robot_to_eff" type="fixed">
@@ -19,10 +19,10 @@
         <child link="base_link" />
         <origin xyz="0.0 0.0 0.0" rpy="0.0 0.0 0.0" />
-    </joint> -->
+    </joint>
     <joint name="world_to_camera" type="fixed">
         <parent link="world" />
         <child link="camera_frame" />
         <origin xyz="-0.25 -0.5 1.25" rpy="0.0 3.14159 0.0" />
-    </joint>
+    </joint> -->
     </xacro:macro>
 </robot>

Commit message: Updated with initial Gazebo simulations

File: abb_irb2600_trispector_support/urdf/abb_irb2600_trispector_macro.xacro (robot description, xacro)
@@ -4,13 +4,13 @@
     <xacro:include filename="$(find abb_irb2600_support)/urdf/irb2600_12_165_macro.xacro" />
     <xacro:include filename="$(find trispector_1060_support)/urdf/trispector_macro.xacro" />
-    <xacro:abb_irb2600_12_165 prefix="" />
-    <xacro:trispector prefix="" />
+    <xacro:abb_irb2600_12_165 prefix="${prefix}" />
+    <xacro:trispector prefix="${prefix}" />
 <!-- Links -->
     <!-- <link name="world" />
     <link name="camera_frame" /> -->
 <!-- Joints -->
-    <joint name="robot_to_eff" type="fixed">
-        <parent link="tool0" />
-        <child link="eff_frame" />
+    <joint name="${prefix}robot_to_eff" type="fixed">
+        <parent link="${prefix}tool0" />
+        <child link="${prefix}eff_frame" />
         <origin xyz="0.0 0.0 0.0" rpy="-1.5708 -1.5708 0.0" />
     </joint>

File: myworkcell_support/urdf/workcell.urdf (robot description, URDF)
Before this commit: robot myworkcell, 16 links, 15 joints
Links:
- removed link ee_base
- removed link ee_mount
- removed link grinder_frame
- removed link part
- removed link tool1
- added link eff_frame
- added link flange
- added link laser_area, mass 0.1; collision box size=0.001 0.001 0.001; visual mesh filename=package://trispector_1060_support/meshes/visual/trispector_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
- added link scan_area, mass 0.1; collision box size=0.001 0.001 0.001; visual mesh filename=package://trispector_1060_support/meshes/visual/trispector_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
- added link scan_area_origin
- added link tcp
- added link trispector, mass 0.1; collision mesh filename=package://trispector_1060_support/meshes/collision/trispect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; visual mesh filename=package://trispector_1060_support/meshes/visual/trispector_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
- link base_link: mass None -> 0.1
- link link_1: mass None -> 0.1
- link link_2: mass None -> 0.1
- link link_3: mass None -> 0.1
- link link_4: mass None -> 0.1
- link link_5: mass None -> 0.1
- link link_6: mass None -> 0.1
Joints:
- removed joint ee_base-tool1
- removed joint ee_mount-ee_base
- removed joint joint6-tool0
- removed joint tool1-part
- removed joint tool_to_puzzle
- removed joint world_to_grinder
- added joint eff_frame_to_trispector: type fixed, parent eff_frame, child trispector, origin xyz=0.0 0.0 0.0 rpy=0.0 0.0 0.0
- added joint joint_6-flange: type fixed, parent link_6, child flange, origin xyz=0 0 0 rpy=0 0 0
- added joint joint_scan_area_origin: type fixed, parent tcp, child scan_area_origin, origin xyz=0.149 0.0 -0.04225 rpy=-1.5708 0 -1.5708
- added joint joint_tcp: type fixed, parent trispector, child tcp, origin xyz=0.088 0.0 0.075 rpy=1.5708 0 1.5708
- added joint link_6-tool0: type fixed, parent flange, child tool0, origin xyz=0 0 0 rpy=0 1.57079632679 0
- added joint origin_to_laser_area: type fixed, parent scan_area_origin, child laser_area, origin xyz=0.0 0.0 0.0 rpy=0.0 0.0 0.0
- added joint origin_to_scan_area: type fixed, parent scan_area_origin, child scan_area, origin xyz=0.0 0.0 0.0 rpy=0.0 0.0 0.0
- added joint robot_to_eff: type fixed, parent tool0, child eff_frame, origin xyz=0.0 0.0 0.0 rpy=-1.5708 -1.5708 0.0

File: myworkcell_support/urdf/workcell.xacro (robot description, xacro)
@@ -31,5 +31,6 @@
     <origin xyz="0 0 0" rpy="1.5708 0 0"/>
   </joint>
-  <!-- <joint name="robot_to_eff" type="fixed">
+<!--
+  <joint name="robot_to_eff" type="fixed">
     <parent link="tool0" />
     <child link="eff_frame" />

File: trispector_1060_support/urdf/trispector_macro.xacro (robot description, xacro)
@@ -2,4 +2,8 @@
 <robot xmlns:xacro="http://ros.org/wiki/xacro">
     <xacro:macro name="trispector" params="prefix">
+    <xacro:macro name="inertia_formula" params="x y z mass">
+        <mass value="${mass}" />
+        <inertia ixx="${0.0833333 * mass * (y*y + z*z)}" ixy="0.0" ixz="0.0" iyy="${0.0833333 * mass * (x*x + z*z)}" iyz="0.0" izz="${0.0833333 * mass * (x*x + y*y)}" />
+    </xacro:macro>
     <!-- Links -->
     <link name="${prefix}eff_frame"/>
@@ -20,5 +24,10 @@
             </geometry>
         </collision>
-        <inertia ixx="0.0" ixy="0.0" ixz="0.0" iyy="0.0" iyz="0.0" izz="0.0" />
+        <inertial>
+            <origin rpy="0 0 0" xyz="0.043727 0.000030 0.073270" />
+            <!-- <xacro:inertia_formula mass="1.9" x="0.1" y="0.325" z="0.1" /> -->
+            <mass value="1.9" />
+            <inertia ixx="0.0204453777545" ixy="0" ixz="0" iyy="0.0057875650741" iyz="0" izz="0.0171436334722" />
+        </inertial>
     </link>
     <joint name="${prefix}eff_frame_to_trispector" type="fixed">
@@ -35,5 +44,5 @@
     <link name="${prefix}scan_area_origin" type="fixed" />
     <joint name="${prefix}joint_scan_area_origin" type="fixed">
-        <origin xyz="0.149 0.0 -0.04225" rpy="-1.5708 0 -1.5708" />
+        <origin xyz="-0.085 0.0 -0.045" rpy="-1.5708 -1.5708 -1.5708" /> <!-- 22.64 deg // 0.39514254 rad -->
         <parent link="${prefix}tcp" />
         <child link="${prefix}scan_area_origin" />
@@ -43,43 +52,43 @@
             <origin xyz="0 0 0" rpy="0 0 0" />
             <geometry>
-              <mesh filename="package://trispector_1060_support/meshes/visual/trispector_scan_area.stl" />
+                <box size="0.001 0.001 0.001"/>
             </geometry>
-            <material name="Grey">
-              <color rgba="235.0 235.0 235.0 0.3" />
-            </material>
         </visual>
-        <collision>
+        <!-- <collision>
+            <origin xyz="0 0.5 0" rpy="0 0 0" />
+            <geometry>
+                <box size="0.001 0.001 0.001"/>
+            </geometry>
+        </collision> -->
+        <!-- <inertia ixx="0.0" ixy="0.0" ixz="0.0" iyy="0.0" iyz="0.0" izz="0.0" /> -->
+    </link>
+    <link name="${prefix}laser_area_origin" type="fixed" />
+    <joint name="${prefix}joint_laser_area_origin" type="fixed">
+        <origin xyz="0.135 0.0 -0.045" rpy="-1.5708 -1.5708 -1.5708" />
+        <parent link="${prefix}tcp" />
+        <child link="${prefix}laser_area_origin" />
+    </joint>
+    <link name="${prefix}laser_area">
+        <visual>
             <origin xyz="0 0 0" rpy="0 0 0" />
             <geometry>
                 <box size="0.001 0.001 0.001"/>
             </geometry>
-        </collision>
-        <inertia ixx="0.0" ixy="0.0" ixz="0.0" iyy="0.0" iyz="0.0" izz="0.0" />
-    </link>
-    <link name="${prefix}laser_area">
-        <visual>
-            <origin xyz="0 0 0" rpy="0 0 0" />
-            <geometry>
-              <mesh filename="package://trispector_1060_support/meshes/visual/trispector_laser_area.stl" />
-            </geometry>
-            <material name="Red">
-              <color rgba="200.0 0.0 0.0 0.4" />
-            </material>
         </visual>
-        <collision>
-            <origin xyz="0 0 0" rpy="0 0 0" />
+        <!-- <collision>
+            <origin xyz="0 0 0.05" rpy="0 0 0" />
             <geometry>
                 <box size="0.001 0.001 0.001"/>
             </geometry>
-        </collision>
-        <inertia ixx="0.0" ixy="0.0" ixz="0.0" iyy="0.0" iyz="0.0" izz="0.0" />
+        </collision> -->
+        <!-- <inertia ixx="0.0" ixy="0.0" ixz="0.0" iyy="0.0" iyz="0.0" izz="0.0" /> -->
     </link>
     <joint name="${prefix}origin_to_scan_area" type="fixed">
         <parent link="scan_area_origin" />
         <child link="scan_area" />
-        <origin xyz="0.0 0.0 0.0" rpy="0.0 0.0 0.0" />
+        <origin xyz="0.0 0.0 0.0" rpy="0.0 -0.3951 0.0" />
     </joint>
     <joint name="${prefix}origin_to_laser_area" type="fixed">
-        <parent link="scan_area_origin" />
+        <parent link="laser_area_origin" />
         <child link="laser_area" />
         <origin xyz="0.0 0.0 0.0" rpy="0.0 0.0 0.0" />
