Commit message: Separated abb_irb2600_gazebo_support

File: abb_irb2600_gazebo/urdf/irb2600_12_165_macro.xacro (robot description, xacro)
@@ -1,5 +1,5 @@
 <?xml version="1.0"?>
 <robot xmlns:xacro="http://ros.org/wiki/xacro">
-    <xacro:include filename="$(find abb_irb2600_support)/urdf/irb2600_12_165_macro.xacro" />
+    <xacro:include filename="$(find abb_irb2600_gazebo_support)/urdf/irb2600_12_165_macro.xacro" />
     <xacro:macro name="abb_irb2600_12_165_gazebo" params="prefix">
         <!-- get base ABB IRB2600 model -->

File: abb_irb2600_gazebo/urdf/tmp.urdf (robot description, URDF)
Before this commit: robot abb_irb2600_12_165_gazebo, 11 links, 10 joints
Links:
- link base_link: geometry collision mesh filename=package://abb_irb2600_gazebo_support/meshes/irb2600_12_165/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; visual mesh filename=package://abb_irb2600_gazebo_support/meshes/irb2600_12_165/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
- link link_1: geometry collision mesh filename=package://abb_irb2600_gazebo_support/meshes/irb2600_12_165/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; visual mesh filename=package://abb_irb2600_gazebo_support/meshes/irb2600_12_165/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
- link link_2: geometry collision mesh filename=package://abb_irb2600_gazebo_support/meshes/irb2600_12_165/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; visual mesh filename=package://abb_irb2600_gazebo_support/meshes/irb2600_12_165/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
- link link_3: geometry collision mesh filename=package://abb_irb2600_gazebo_support/meshes/irb2600_12_165/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; visual mesh filename=package://abb_irb2600_gazebo_support/meshes/irb2600_12_165/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
- link link_4: geometry collision mesh filename=package://abb_irb2600_gazebo_support/meshes/irb2600_12_165/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; visual mesh filename=package://abb_irb2600_gazebo_support/meshes/irb2600_12_165/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
- link link_5: geometry collision mesh filename=package://abb_irb2600_gazebo_support/meshes/irb2600_12_165/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; visual mesh filename=package://abb_irb2600_gazebo_support/meshes/irb2600_12_165/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
- link link_6: geometry collision mesh filename=package://abb_irb2600_gazebo_support/meshes/irb2600_12_165/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; visual mesh filename=package://abb_irb2600_gazebo_support/meshes/irb2600_12_165/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

File: abb_irb2600_trispector_gazebo/urdf/tmp.urdf (robot description, URDF)
Before this commit: robot abb_irb2600_trispector_gazebo, 17 links, 16 joints
Links:
- link base_link: geometry collision mesh filename=package://abb_irb2600_gazebo_support/meshes/irb2600_12_165/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; visual mesh filename=package://abb_irb2600_gazebo_support/meshes/irb2600_12_165/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
- link link_1: geometry collision mesh filename=package://abb_irb2600_gazebo_support/meshes/irb2600_12_165/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; visual mesh filename=package://abb_irb2600_gazebo_support/meshes/irb2600_12_165/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
- link link_2: geometry collision mesh filename=package://abb_irb2600_gazebo_support/meshes/irb2600_12_165/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; visual mesh filename=package://abb_irb2600_gazebo_support/meshes/irb2600_12_165/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
- link link_3: geometry collision mesh filename=package://abb_irb2600_gazebo_support/meshes/irb2600_12_165/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; visual mesh filename=package://abb_irb2600_gazebo_support/meshes/irb2600_12_165/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
- link link_4: geometry collision mesh filename=package://abb_irb2600_gazebo_support/meshes/irb2600_12_165/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; visual mesh filename=package://abb_irb2600_gazebo_support/meshes/irb2600_12_165/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
- link link_5: geometry collision mesh filename=package://abb_irb2600_gazebo_support/meshes/irb2600_12_165/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; visual mesh filename=package://abb_irb2600_gazebo_support/meshes/irb2600_12_165/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
- link link_6: geometry collision mesh filename=package://abb_irb2600_gazebo_support/meshes/irb2600_12_165/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; visual mesh filename=package://abb_irb2600_gazebo_support/meshes/irb2600_12_165/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

File: abb_irb2600_trispector_on_track_support/urdf/gazebo_abb_irb2600_trispector_on_track.urdf (robot description, URDF)
Before this commit: robot abb_irb2600_trispector_on_track, 22 links, 21 joints
Links:
- link base_link: geometry collision mesh filename=package://abb_irb2600_gazebo_support/meshes/irb2600_12_165/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; visual mesh filename=package://abb_irb2600_gazebo_support/meshes/irb2600_12_165/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
- link link_1: geometry collision mesh filename=package://abb_irb2600_gazebo_support/meshes/irb2600_12_165/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; visual mesh filename=package://abb_irb2600_gazebo_support/meshes/irb2600_12_165/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
- link link_2: geometry collision mesh filename=package://abb_irb2600_gazebo_support/meshes/irb2600_12_165/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; visual mesh filename=package://abb_irb2600_gazebo_support/meshes/irb2600_12_165/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
- link link_3: geometry collision mesh filename=package://abb_irb2600_gazebo_support/meshes/irb2600_12_165/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; visual mesh filename=package://abb_irb2600_gazebo_support/meshes/irb2600_12_165/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
- link link_4: geometry collision mesh filename=package://abb_irb2600_gazebo_support/meshes/irb2600_12_165/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; visual mesh filename=package://abb_irb2600_gazebo_support/meshes/irb2600_12_165/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
- link link_5: geometry collision mesh filename=package://abb_irb2600_gazebo_support/meshes/irb2600_12_165/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; visual mesh filename=package://abb_irb2600_gazebo_support/meshes/irb2600_12_165/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
- link link_6: geometry collision mesh filename=package://abb_irb2600_gazebo_support/meshes/irb2600_12_165/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; visual mesh filename=package://abb_irb2600_gazebo_support/meshes/irb2600_12_165/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

File: abb_irb2600_trispector_support/urdf/abb_irb2600_trispector_macro.xacro (robot description, xacro)
@@ -2,5 +2,5 @@
 <robot xmlns:xacro="http://ros.org/wiki/xacro">
     <xacro:macro name="abb_irb2600_trispector" params="prefix">
-    <xacro:include filename="$(find abb_irb2600_support)/urdf/irb2600_12_165_macro.xacro" />
+    <xacro:include filename="$(find abb_irb2600_gazebo_support)/urdf/irb2600_12_165_macro.xacro" />
     <xacro:include filename="$(find trispector_1060_support)/urdf/trispector_macro.xacro" />
     <xacro:abb_irb2600_12_165 prefix="${prefix}" />

File: myworkcell_support/urdf/workcell.urdf (robot description, URDF)
Before this commit: robot myworkcell, 18 links, 17 joints
Links:
- link base_link: geometry collision mesh filename=package://abb_irb2600_gazebo_support/meshes/irb2600_12_165/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; visual mesh filename=package://abb_irb2600_gazebo_support/meshes/irb2600_12_165/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
- link link_1: geometry collision mesh filename=package://abb_irb2600_gazebo_support/meshes/irb2600_12_165/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; visual mesh filename=package://abb_irb2600_gazebo_support/meshes/irb2600_12_165/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
- link link_2: geometry collision mesh filename=package://abb_irb2600_gazebo_support/meshes/irb2600_12_165/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; visual mesh filename=package://abb_irb2600_gazebo_support/meshes/irb2600_12_165/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
- link link_3: geometry collision mesh filename=package://abb_irb2600_gazebo_support/meshes/irb2600_12_165/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; visual mesh filename=package://abb_irb2600_gazebo_support/meshes/irb2600_12_165/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
- link link_4: geometry collision mesh filename=package://abb_irb2600_gazebo_support/meshes/irb2600_12_165/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; visual mesh filename=package://abb_irb2600_gazebo_support/meshes/irb2600_12_165/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
- link link_5: geometry collision mesh filename=package://abb_irb2600_gazebo_support/meshes/irb2600_12_165/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; visual mesh filename=package://abb_irb2600_gazebo_support/meshes/irb2600_12_165/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
- link link_6: geometry collision mesh filename=package://abb_irb2600_gazebo_support/meshes/irb2600_12_165/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; visual mesh filename=package://abb_irb2600_gazebo_support/meshes/irb2600_12_165/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

File: myworkcell_support/urdf/workcell.xacro (robot description, xacro)
@@ -1,5 +1,5 @@
 <?xml version="1.0" ?>
 <robot name="myworkcell" xmlns:xacro="http://ros.org/wiki/xacro">
-  <xacro:include filename="$(find abb_irb2600_support)/urdf/irb2600_12_165_macro.xacro" />
+  <xacro:include filename="$(find abb_irb2600_gazebo_support)/urdf/irb2600_12_165_macro.xacro" />
   <!-- <xacro:include filename="$(find trispector_1060_support)/urdf/trispector_macro.xacro" /> -->
   <xacro:include filename="$(find myworkcell_support)/urdf/grinder.xacro" />
